File: AMineralFire/MineralFire.brd (EAGLE design)
At the start: 160 x 100 mm, 77 parts, among them IC1 LM358, IC2 OP-AMP, Q1 20MHz, Q2 20MHz, Q3 2N3906, Q4 2N3906, Q5 2N3906, Q6 2N3906, Q7 2N3906, Q8 2N3906, Q9 2N3906, T1 200mA/40V, T2 200mA/40V, T3 200mA/40V, T4 200mA/40V, T5 200mA/40V, U1 328P, U2 328P, U3 +12v

Commit message: Moving atmega to smd
Parts:
- added U4: ATMEGA328P_TQFP, SparkFun-IC-Microcontroller:TQFP32-08
Connections:
- net MISO2: now also U4.15, U4.16; no longer U2.18
- net SCK2: now also U4.17; no longer U2.19
Changed lines of the file:
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@@
 <attribute name="PROD_ID" value="NA-XXXXX" x="64.77" y="78.74" size="1.778" layer="27" display="off"/>
+</element>
+<element name="U4" library="SparkFun-IC-Microcontroller" package="TQFP32-08" value="ATMEGA328P_TQFP" x="-101.6" y="0">
+<attribute name="PROD_ID" value="IC-09069" x="-101.6" y="0" size="1.778" layer="27" display="off"/>
 </element>
 </elements>
@@
 </signal>
 <signal name="SCK2">
-<contactref element="U2" pad="19"/>
 <contactref element="ISP2" pad="3"/>
-<wire x1="36.83" y1="90.17" x2="-26.67" y2="73.66" width="0" layer="19" extent="1-1"/>
+<contactref element="U4" pad="17"/>
+<wire x1="-97.3074" y1="-2.8" x2="36.83" y2="90.17" width="0" layer="19" extent="1-1"/>
 </signal>
 <signal name="MISO2">
-<contactref element="U2" pad="18"/>
 <contactref element="ISP2" pad="1"/>
-<wire x1="34.29" y1="90.17" x2="-24.13" y2="73.66" width="0" layer="19" extent="1-1"/>
+<contactref element="U4" pad="15"/>
+<contactref element="U4" pad="16"/>
+<wire x1="-98.8" y1="-4.2926" x2="34.29" y2="90.17" width="0" layer="19" extent="1-1"/>
+<wire x1="-99.6" y1="-4.2926" x2="-98.8" y2="-4.2926" width="0" layer="19" extent="1-1"/>
 </signal>
 <signal name="MOSI2">

Commit message: moving to SMD
Parts:
- removed C1, C2: 22pF, SparkFun-Capacitors:0603
- removed IC1: LM358, SparkFun-IC-Amplifiers:DIP08
- removed Q1: 20MHz, adafruit:HC49UP
- removed U1, U2: 328P, SparkFun-IC-Microcontroller:DIP28
- removed V1: 7432N, 74ttl-din:DIL14
- added C14, C15: 22pF, SparkFun-Capacitors:0603
- added IC3: 7432D, 74xx-us:SO14
- added Q10: 20MHz, adafruit:HC49UP
- added U5: ATMEGA328P_TQFP, SparkFun-IC-Microcontroller:TQFP32-08
- C6: device rcl:C075-032X103 -> rcl:C01005
- D1, D2: value 200mA/100V/1V -> 250mA/100V; device SparkFun-DiscreteSemi:DIODE-1N4148 -> SparkFun-DiscreteSemi:SOD-323
- Q3, Q4, Q5, Q6, Q7, Q8, Q9: value 2N3906 -> 200mA/40V; device transistor-pnp:TO92 -> SparkFun-DiscreteSemi:SOT23-3
- R5, R9: device SparkFun-Resistors:AXIAL-0.3 -> SparkFun-Resistors:0603
- T1, T2, T3, T4, T5: value 200mA/40V -> 600mA/40V; device SparkFun-DiscreteSemi:TO-92 -> SparkFun-DiscreteSemi:SOT23-3
- moved R9 187.2 mm to (108.0, 40.6)
- moved R21 176.0 mm to (92.7, 5.08)
- moved R14 167.7 mm to (91.4, 14.0)
- moved R27 164.7 mm to (88.9, 36.8)
- moved R20 164.6 mm to (91.4, 8.89)
- moved R15 161.4 mm to (88.9, 40.6)
- moved R10 153.3 mm to (47.0, 15.2)
- moved R3 149.9 mm to (68.6, 92.7)
- moved MODESW3 143.1 mm to (78.7, 12.7), turned to 270 degrees
- moved C12 141.3 mm to (62.2, 36.8)
- moved R2 140.0 mm to (68.6, 88.9)
- moved R6 138.5 mm to (71.1, 17.8)
- moved R5 137.4 mm to (71.1, 7.62)
- moved D2 134.4 mm to (92.7, 81.3)
- moved D1 133.3 mm to (101.6, 80.0)
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Connections:
- removed net CS: U1.16
- removed net N$1: C1.1, Q1.2, U1.9
- removed net N$2: C2.1, Q1.1, U1.10
- new net N$21: C14.1, Q10.2, U5.7
- new net N$22: C15.1, Q10.1, U5.8
- new net RST2: ISP2.5, U4.29
- net +12V: now also IC2.8; no longer IC1.8
- net +5V: now also IC3.14, Q3.2, Q4.2, Q5.2, Q6.2, Q7.2, Q8.2, Q9.2, R5.1, R9.2, U4.18, U4.20, U4.4, U4.6, U5.18, U5.20, U5.4, U5.6; no longer Q3.3, Q4.3, Q5.3, Q6.3, Q7.3, Q8.3, Q9.3, R5.P$1, R9.P$2, U1.20, U1.21, U1.7, U2.20, U2.21, U2.7, V1.14
- net B_TRIG: now also R9.1, U5.1; no longer R9.P$1, U1.5
- net C-DIG1: now also T2.1, U4.13; no longer T2.2, U2.15
- net C-DIG2: now also T3.1, U4.25; no longer T3.2, U2.25
- net C-DIG3: now also T4.1, U4.26; no longer T4.2, U2.26
- net C-DIG4: now also T5.1, U4.1; no longer T5.2, U2.5
- net C-SEGA: now also Q5.1, U4.23; no longer Q5.2, U2.23
- net C-SEGB: now also Q9.1, U4.32; no longer Q9.2, U2.4
- net C-SEGC: now also Q7.1, U4.12; no longer Q7.2, U2.14
- net C-SEGD: now also Q3.1, U4.10; no longer Q3.2, U2.12
- net C-SEGDP: now also U4.9; no longer U2.11
- net C-SEGE: now also Q4.1, U4.11; no longer Q4.2, U2.13
- net C-SEGF: now also Q8.1, U4.24; no longer Q8.2, U2.24
- net C-SEGG: now also Q6.1, U4.2; no longer Q6.2, U2.6
- net GND: now also C14.2, C15.2, IC3.7, T1.2, T2.2, T3.2, T4.2, T5.2, U4.21, U4.3, U4.5, U5.21, U5.3, U5.5; no longer C1.2, C2.2, IC1.4, T1.1, T2.1, T3.1, T4.1, T5.1, U1.22, U1.8, U2.22, U2.8, V1.7
- net LBUTTON: now also IC3.2; no longer V1.2
- net LTRIG: now also IC3.1; no longer V1.1
- net MISO: now also U5.16; no longer U1.18
- net MISO2: no longer U4.15
- net MOSI: now also U5.15; no longer U1.17
- net MOSI2: now also U4.15; no longer U2.16, U2.17
- net N$11: now also Q3.3; no longer Q3.1
- net N$13: now also Q9.3; no longer Q9.1
- net N$14: now also Q8.3; no longer Q8.1
- net N$15: now also T1.1; no longer T1.2
- net N$16: now also Q7.3; no longer Q7.1
- net N$17: now also Q6.3; no longer Q6.1
- net N$20: now also Q5.3; no longer Q5.1
- net N$5: now also Q4.3; no longer Q4.1
- net N$7: now also U4.7; no longer U2.9
- net N$8: now also U4.8; no longer U2.10
- net RST: now also U5.29; no longer ISP2.5, U1.1, U2.1
- net SCK: now also U5.17; no longer U1.19
- net SCL: now also U4.28, U5.28; no longer U1.28, U2.28
- net SDA: now also U4.27, U5.27; no longer U1.27, U2.27
- net T1: now also U5.9; no longer U1.11
- net T2: now also U5.2; no longer U1.6
- net T3: now also U5.25; no longer U1.25
- net T4: now also U5.26; no longer U1.26
- net T5: now also R5.2, U5.23; no longer R5.P$2, U1.23
- net T6: now also U5.24; no longer U1.24
- net T7: now also U5.10; no longer U1.12
- net T8: now also U5.11; no longer U1.13
- net TRIG: now also IC3.3, U5.32; no longer U1.4, V1.3
- net TRIGO: now also U5.12; no longer U1.14
Other:
- board size 160 x 100 mm -> 110.5 x 100 mm

Commit message: first SMD
Parts:
- moved ISP2 58.4 mm to (7.62, 69.8)
- moved ISP1 48.7 mm to (85.1, 43.2), turned to 0 degrees
- moved R9 34.5 mm to (73.7, 36.8)
- moved C4 34.2 mm to (72.4, 52.1)
- moved BUT1 29.9 mm to (71.1, 26.7), flipped to the bottom
- moved BUT 29.2 mm to (71.1, 44.5), flipped to the bottom
- moved D1 26.4 mm to (80.0, 64.8)
- moved IC3 25.5 mm to (54.6, 26.7)
- moved POWER 25.2 mm to (80.0, 71.1), turned to 270 degrees
- moved R21 22.9 mm to (69.8, 5.08)
- moved C5 22.2 mm to (72.4, 57.1)
- moved PROGSW 21.7 mm to (80.0, 10.2)
- moved R14 21.6 mm to (69.8, 15.2)
- moved R20 21.6 mm to (69.8, 10.2)
- moved R15 20.5 mm to (68.6, 38.1), turned to 180 degrees
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Other:
- board size 110.5 x 100 mm -> 91.4 x 77.1 mm

Commit message: routing
Routing:
- net GND: track 0.00 -> 407.0 mm, vias 0 -> 7
- net +5V: track 0.00 -> 327.4 mm, vias 0 -> 14
- net -12V: track 0.00 -> 139.4 mm, vias 0 -> 2
- net +12V: track 0.00 -> 98.7 mm, vias 0 -> 4
- net TRIGO: track 0.00 -> 94.8 mm, vias 0 -> 1
- net T5: track 0.00 -> 65.0 mm, vias 0 -> 1
- net T7: track 0.00 -> 61.6 mm, vias 0 -> 1
- net T8: track 0.00 -> 57.7 mm, vias 0 -> 1
- net SCL: track 0.00 -> 54.3 mm, vias 0 -> 4
- net T3: track 0.00 -> 51.7 mm
- net SDA: track 0.00 -> 51.4 mm, vias 0 -> 4
- net T2: track 0.00 -> 50.2 mm, vias 0 -> 1
- net RST: track 0.00 -> 45.6 mm, vias 0 -> 2
- net B_TRIG: track 0.00 -> 41.0 mm, vias 0 -> 1
- net T6: track 0.00 -> 40.0 mm, vias 0 -> 3
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