File: AMineralFire/MineralFire.brd (EAGLE design)
At the start: 109.9 x 77 mm, 77 parts, among them IC1 LM358, Q1 20MHz, Q2 20MHz, Q3 2N3906, Q4 2N3906, Q5 2N3906, Q6 2N3906, Q7 2N3906, Q8 2N3906, Q9 2N3906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

Commit message: added diode to switch
Parts:
- added D4: 200mA/100V/1V, SparkFun-DiscreteSemi:DIODE-1N4148
- R27: value 10k -> 100; device SparkFun-Resistors:AXIAL-0.3 -> SparkFun-Resistors:AXIAL-0.3EZ
- moved R27 12.8 mm to (61.0, 7.62)
Connections:
- new net N$21: BUT1.3, BUT1.4, BUT1.A, D4.A
- net +5V: now also BUT1.1, BUT1.2; no longer R27.P$2
- net BUTLED: no longer BUT1.A
- net GND: now also R27.P$1; no longer BUT1.3, BUT1.4
- net LBUTTON: now also D4.C, R27.P$2; no longer BUT1.1, BUT1.2, R27.P$1
Routing:
- net LBUTTON: track 58.9 -> 51.6 mm
- net GND: track 496.6 -> 489.7 mm
- net N$21: track 0.00 -> 6.91 mm
- net +5V: track 400.9 -> 405.5 mm
Changed lines of the file:
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@@
 <attribute name="VALUE" value="100" x="6.35" y="2.54" size="1.778" layer="27" display="off"/>
-</element>
-<element name="R27" library="SparkFun-Resistors" package="AXIAL-0.3" value="10k" x="62.23" y="20.32" rot="R90">
-<attribute name="PROD_ID" value="RES-12183" x="62.23" y="20.32" size="1.778" layer="27" rot="R90" display="off"/>
 </element>
 <element name="R30" library="SparkFun-Resistors" package="AXIAL-0.3" value="330" x="105.41" y="17.78" rot="R90">
@@
 </element>
 <element name="V1" library="74ttl-din" library_urn="urn:adsk.eagle:library:84" package="DIL14" value="7409N" x="49.53" y="20.32"/>
+<element name="D4" library="SparkFun-DiscreteSemi" package="DIODE-1N4148" value="200mA/100V/1V" x="62.23" y="20.32" rot="R270">
+<attribute name="PROD_ID" value="DIO-08378" x="62.23" y="20.32" size="1.778" layer="27" rot="R270" display="off"/>
+</element>
+<element name="R27" library="SparkFun-Resistors" package="AXIAL-0.3EZ" value="100" x="60.96" y="7.62" rot="R90">
+<attribute name="PROD_ID" value="RES-12181" x="60.96" y="7.62" size="1.778" layer="27" rot="R90" display="off"/>
+</element>
 </elements>
 <signals>
@@
 <contactref element="T4" pad="1"/>
 <contactref element="T5" pad="1"/>
-<contactref element="BUT1" pad="3"/>
-<contactref element="BUT1" pad="4"/>
 <contactref element="R30" pad="P$1"/>
 <contactref element="V1" pad="7"/>
@@
 <wire x1="56.9976" y1="16.1544" x2="57.15" y2="16.51" width="0.8" layer="16"/>
 <wire x1="40.6908" y1="7.62" x2="40.64" y2="7.62" width="0.8" layer="16"/>
-<wire x1="92.964" y1="14.0208" x2="92.7354" y2="14.0208" width="0.8" layer="1"/>
-<wire x1="94.6404" y1="15.6972" x2="92.964" y2="14.0208" width="0.8" layer="1"/>
-<wire x1="94.6404" y1="17.2974" x2="94.6404" y2="15.6972" width="0.8" layer="1"/>
-<wire x1="92.8878" y1="19.05" x2="94.6404" y2="17.2974" width="0.8" layer="1"/>
-<wire x1="92.71" y1="19.05" x2="92.8878" y2="19.05" width="0.8" layer="1"/>
-<wire x1="92.7354" y1="14.0208" x2="92.71" y2="13.97" width="0.8" layer="1"/>
 <wire x1="95.25" y1="21.5646" x2="97.7646" y2="21.5646" width="0.8" layer="16"/>
 <wire x1="92.7354" y1="19.05" x2="95.25" y2="21.5646" width="0.8" layer="16"/>
 <wire x1="97.7646" y1="21.5646" x2="97.79" y2="21.59" width="0.8" layer="16"/>
-<wire x1="92.7354" y1="19.05" x2="92.71" y2="19.05" width="0.8" layer="16"/>
 <wire x1="99.06" y1="28.8036" x2="99.06" y2="30.48" width="0.8" layer="16"/>
 <wire x1="97.536" y1="27.2796" x2="99.06" y2="28.8036" width="0.8" layer="16"/>
@@
 <via x="20.2692" y="8.3058" extent="1-16" drill="0.35"/>
 <via x="66.294" y="42.2148" extent="1-16" drill="0.35"/>
+<contactref element="R27" pad="P$1"/>
 <wire x1="48.768" y1="6.096" x2="53.34" y2="1.12" width="0" layer="19" extent="16-16"/>
+<wire x1="60.96" y1="3.81" x2="15.8496" y2="3.5814" width="0" layer="19" extent="16-16"/>
 </signal>
 <signal name="RST">
@@
 <contactref element="Q4" pad="3"/>
 <contactref element="U3" pad="OUT"/>
-<contactref element="R27" pad="P$2"/>
 <contactref element="V1" pad="14"/>
 <wire x1="24.6888" y1="72.39" x2="24.13" y2="72.39" width="0.8" layer="16"/>
@@
 <wire x1="63.4746" y1="22.86" x2="66.04" y2="22.86" width="0.8" layer="1"/>
 <wire x1="62.2554" y1="24.0792" x2="63.4746" y2="22.86" width="0.8" layer="1"/>
-<wire x1="62.2554" y1="24.0792" x2="62.23" y2="24.13" width="0.8" layer="1"/>
 <wire x1="67.6656" y1="24.384" x2="77.4954" y2="24.384" width="0.8" layer="1"/>
 <wire x1="66.3702" y1="23.0886" x2="67.6656" y2="24.384" width="0.8" layer="1"/>
@@
 <wire x1="50.7492" y1="29.337" x2="54.3306" y2="29.337" width="0.8" layer="1"/>
 <wire x1="49.911" y1="30.1752" x2="50.7492" y2="29.337" width="0.8" layer="1"/>
-<wire x1="61.8744" y1="24.3078" x2="62.23" y2="24.13" width="0.8" layer="1"/>
 <wire x1="49.911" y1="30.1752" x2="49.53" y2="30.353" width="0.8" layer="1"/>
 <wire x1="57.6072" y1="50.8254" x2="57.0738" y2="50.8254" width="0.8" layer="1"/>
@@
 <via x="59.2074" y="52.4256" extent="1-16" drill="0.35"/>
 <via x="57.531" y="74.5236" extent="1-16" drill="0.35"/>
+<contactref element="BUT1" pad="2"/>
+<contactref element="BUT1" pad="1"/>
+<wire x1="87.63" y1="19.05" x2="87.63" y2="13.97" width="0.1524" layer="1"/>
+<wire x1="95.0214" y1="23.0886" x2="87.63" y2="19.05" width="0" layer="19" extent="1-1"/>
+<wire x1="62.2554" y1="24.0792" x2="61.8744" y2="24.3078" width="0" layer="19" extent="1-1"/>
 </signal>
 <signal name="MISO">
@@
 </signal>
 <signal name="LBUTTON">
-<contactref element="R27" pad="P$1"/>
-<contactref element="BUT1" pad="2"/>
-<contactref element="BUT1" pad="1"/>
 <contactref element="V1" pad="2"/>
-<wire x1="87.63" y1="19.05" x2="87.63" y2="13.97" width="0.1524" layer="1"/>
 <wire x1="45.1104" y1="16.4592" x2="44.5008" y2="16.4592" width="0.1524" layer="1"/>
 <wire x1="46.6344" y1="14.9352" x2="45.1104" y2="16.4592" width="0.1524" layer="1"/>
 <wire x1="60.6552" y1="14.9352" x2="46.6344" y2="14.9352" width="0.1524" layer="1"/>
-<wire x1="62.23" y1="16.51" x2="60.6933" y2="14.9733" width="0.1524" layer="1"/>
 <wire x1="60.6933" y1="14.9733" x2="60.6552" y2="14.9352" width="0.1524" layer="1"/>
 <wire x1="44.5008" y1="16.4592" x2="44.45" y2="16.51" width="0.1524" layer="1"/>
@@
 <wire x1="60.7314" y1="12.7254" x2="66.8274" y2="6.6294" width="0.1524" layer="1"/>
 <wire x1="60.7314" y1="14.9352" x2="60.7314" y2="12.7254" width="0.1524" layer="1"/>
-<wire x1="87.63" y1="13.9446" x2="87.63" y2="13.97" width="0.1524" layer="1"/>
 <wire x1="60.7314" y1="14.9352" x2="60.6933" y2="14.9733" width="0.1524" layer="1"/>
+<contactref element="D4" pad="C"/>
+<contactref element="R27" pad="P$2"/>
+<wire x1="62.23" y1="16.51" x2="44.5008" y2="16.4592" width="0" layer="19" extent="1-1"/>
+<wire x1="60.96" y1="11.43" x2="62.23" y2="16.51" width="0" layer="19" extent="1-1"/>
 </signal>
 <signal name="N$7">
@@
 <signal name="BUTLED">
 <contactref element="U1" pad="15"/>
-<contactref element="BUT1" pad="A"/>
 <wire x1="90.1446" y1="15.0876" x2="90.1446" y2="13.8684" width="0.1524" layer="16"/>
 <wire x1="86.487" y1="18.7452" x2="90.1446" y2="15.0876" width="0.1524" layer="16"/>
 <wire x1="86.487" y1="41.8338" x2="86.487" y2="18.7452" width="0.1524" layer="16"/>
 <wire x1="82.6008" y1="45.72" x2="86.487" y2="41.8338" width="0.1524" layer="16"/>
-<wire x1="90.1446" y1="13.8684" x2="90.17" y2="13.81" width="0.1524" layer="16"/>
 <wire x1="82.6008" y1="45.72" x2="82.55" y2="45.72" width="0.1524" layer="16"/>
 </signal>
+<signal name="N$21" class="1">
+<contactref element="BUT1" pad="3"/>
+<contactref element="BUT1" pad="4"/>
+<wire x1="92.964" y1="14.0208" x2="92.7354" y2="14.0208" width="0.8" layer="1"/>
+<wire x1="94.6404" y1="15.6972" x2="92.964" y2="14.0208" width="0.8" layer="1"/>
+<wire x1="94.6404" y1="17.2974" x2="94.6404" y2="15.6972" width="0.8" layer="1"/>
+<wire x1="92.8878" y1="19.05" x2="94.6404" y2="17.2974" width="0.8" layer="1"/>
+<wire x1="92.71" y1="19.05" x2="92.8878" y2="19.05" width="0.8" layer="1"/>
+<wire x1="92.7354" y1="14.0208" x2="92.71" y2="13.97" width="0.8" layer="1"/>
+<contactref element="BUT1" pad="A"/>
+<contactref element="D4" pad="A"/>
+<wire x1="90.17" y1="13.81" x2="92.71" y2="13.97" width="0" layer="19" extent="1-1"/>
+<wire x1="62.23" y1="24.13" x2="90.17" y2="13.81" width="0" layer="19" extent="1-1"/>
+</signal>
 </signals>

Commit message: new input circuit
Parts:
- removed D4: 200mA/100V/1V, SparkFun-DiscreteSemi:DIODE-1N4148
- added R31: 10K, SparkFun-Resistors:AXIAL-0.3EZ
- R27: value 100 -> 10K
Connections:
- net +5V: now also R27.P$2, R31.P$2; no longer BUT1.1, BUT1.2
- net BUTLED: now also BUT1.A
- net GND: no longer R27.P$1
- net LBUTTON: now also BUT1.3, BUT1.4; no longer D4.C, R27.P$2
- net N$21: now also BUT1.1, BUT1.2, R31.P$1; no longer BUT1.3, BUT1.4, BUT1.A, D4.A
- net TRIG: now also R27.P$1
Routing:
- net LBUTTON: track 51.6 -> 58.5 mm
- net +5V: track 405.5 -> 400.4 mm
- net N$21: track 6.91 -> 5.08 mm
Changed lines of the file:
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@@
 <?xml version="1.0" encoding="utf-8"?>
 <!DOCTYPE eagle SYSTEM "eagle.dtd">
-<eagle version="8.2.2">
+<eagle version="8.3.1">
 <drawing>
 <settings>
 <setting alwaysvectorfont="no"/>
+<setting keepoldvectorfont="yes"/>
 <setting verticaltext="up"/>
 </settings>
@@
 </element>
 <element name="V1" library="74ttl-din" library_urn="urn:adsk.eagle:library:84" package="DIL14" value="7409N" x="49.53" y="20.32"/>
-<element name="D4" library="SparkFun-DiscreteSemi" package="DIODE-1N4148" value="200mA/100V/1V" x="62.23" y="20.32" rot="R270">
-<attribute name="PROD_ID" value="DIO-08378" x="62.23" y="20.32" size="1.778" layer="27" rot="R270" display="off"/>
-</element>
-<element name="R27" library="SparkFun-Resistors" package="AXIAL-0.3EZ" value="100" x="60.96" y="7.62" rot="R90">
+<element name="R27" library="SparkFun-Resistors" package="AXIAL-0.3EZ" value="10K" x="60.96" y="7.62" rot="R90">
 <attribute name="PROD_ID" value="RES-12181" x="60.96" y="7.62" size="1.778" layer="27" rot="R90" display="off"/>
+</element>
+<element name="R31" library="SparkFun-Resistors" package="AXIAL-0.3EZ" value="10K" x="80.01" y="19.05">
+<attribute name="PROD_ID" value="RES-12181" x="80.01" y="19.05" size="1.778" layer="27" display="off"/>
 </element>
 </elements>
@@
 <via x="20.2692" y="8.3058" extent="1-16" drill="0.35"/>
 <via x="66.294" y="42.2148" extent="1-16" drill="0.35"/>
-<contactref element="R27" pad="P$1"/>
 <wire x1="48.768" y1="6.096" x2="53.34" y2="1.12" width="0" layer="19" extent="16-16"/>
-<wire x1="60.96" y1="3.81" x2="15.8496" y2="3.5814" width="0" layer="19" extent="16-16"/>
 </signal>
 <signal name="RST">
@@
 <via x="59.2074" y="52.4256" extent="1-16" drill="0.35"/>
 <via x="57.531" y="74.5236" extent="1-16" drill="0.35"/>
-<contactref element="BUT1" pad="2"/>
-<contactref element="BUT1" pad="1"/>
-<wire x1="87.63" y1="19.05" x2="87.63" y2="13.97" width="0.1524" layer="1"/>
-<wire x1="95.0214" y1="23.0886" x2="87.63" y2="19.05" width="0" layer="19" extent="1-1"/>
-<wire x1="62.2554" y1="24.0792" x2="61.8744" y2="24.3078" width="0" layer="19" extent="1-1"/>
+<contactref element="R27" pad="P$2"/>
+<contactref element="R31" pad="P$2"/>
+<wire x1="77.4954" y1="22.86" x2="83.82" y2="19.05" width="0" layer="19" extent="1-1"/>
+<wire x1="61.8744" y1="24.3078" x2="62.2554" y2="24.0792" width="0" layer="19" extent="1-1"/>
+<wire x1="60.96" y1="11.43" x2="63.4746" y2="22.86" width="0" layer="19" extent="1-1"/>
 </signal>
 <signal name="MISO">
@@
 <wire x1="57.15" y1="38.1" x2="53.4924" y2="34.4424" width="0.1524" layer="16"/>
 <wire x1="47.0154" y1="16.5354" x2="46.99" y2="16.51" width="0.1524" layer="16"/>
+<contactref element="R27" pad="P$1"/>
+<wire x1="47.0154" y1="16.5354" x2="60.96" y2="3.81" width="0" layer="19" extent="16-16"/>
 </signal>
 <signal name="B_TRIG">
@@
 <wire x1="60.7314" y1="14.9352" x2="60.7314" y2="12.7254" width="0.1524" layer="1"/>
 <wire x1="60.7314" y1="14.9352" x2="60.6933" y2="14.9733" width="0.1524" layer="1"/>
-<contactref element="D4" pad="C"/>
-<contactref element="R27" pad="P$2"/>
-<wire x1="62.23" y1="16.51" x2="44.5008" y2="16.4592" width="0" layer="19" extent="1-1"/>
-<wire x1="60.96" y1="11.43" x2="62.23" y2="16.51" width="0" layer="19" extent="1-1"/>
+<contactref element="BUT1" pad="3"/>
+<contactref element="BUT1" pad="4"/>
+<wire x1="92.964" y1="14.0208" x2="92.7354" y2="14.0208" width="0.8" layer="1"/>
+<wire x1="94.6404" y1="15.6972" x2="92.964" y2="14.0208" width="0.8" layer="1"/>
+<wire x1="94.6404" y1="17.2974" x2="94.6404" y2="15.6972" width="0.8" layer="1"/>
+<wire x1="92.8878" y1="19.05" x2="94.6404" y2="17.2974" width="0.8" layer="1"/>
+<wire x1="92.71" y1="19.05" x2="92.8878" y2="19.05" width="0.8" layer="1"/>
+<wire x1="92.7354" y1="14.0208" x2="92.71" y2="13.97" width="0.8" layer="1"/>
+<wire x1="87.63" y1="13.9446" x2="92.71" y2="13.97" width="0" layer="19" extent="1-1"/>
 </signal>
 <signal name="N$7">
@@
 <wire x1="82.6008" y1="45.72" x2="86.487" y2="41.8338" width="0.1524" layer="16"/>
 <wire x1="82.6008" y1="45.72" x2="82.55" y2="45.72" width="0.1524" layer="16"/>
+<contactref element="BUT1" pad="A"/>
+<wire x1="90.17" y1="13.81" x2="90.1446" y2="13.8684" width="0" layer="19" extent="16-16"/>
 </signal>
 <signal name="N$21" class="1">
-<contactref element="BUT1" pad="3"/>
-<contactref element="BUT1" pad="4"/>
-<wire x1="92.964" y1="14.0208" x2="92.7354" y2="14.0208" width="0.8" layer="1"/>
-<wire x1="94.6404" y1="15.6972" x2="92.964" y2="14.0208" width="0.8" layer="1"/>
-<wire x1="94.6404" y1="17.2974" x2="94.6404" y2="15.6972" width="0.8" layer="1"/>
-<wire x1="92.8878" y1="19.05" x2="94.6404" y2="17.2974" width="0.8" layer="1"/>
-<wire x1="92.71" y1="19.05" x2="92.8878" y2="19.05" width="0.8" layer="1"/>
-<wire x1="92.7354" y1="14.0208" x2="92.71" y2="13.97" width="0.8" layer="1"/>
-<contactref element="BUT1" pad="A"/>
-<contactref element="D4" pad="A"/>
-<wire x1="90.17" y1="13.81" x2="92.71" y2="13.97" width="0" layer="19" extent="1-1"/>
-<wire x1="62.23" y1="24.13" x2="90.17" y2="13.81" width="0" layer="19" extent="1-1"/>
+<contactref element="BUT1" pad="2"/>
+<contactref element="BUT1" pad="1"/>
+<wire x1="87.63" y1="19.05" x2="87.63" y2="13.97" width="0.1524" layer="1"/>
+<contactref element="R31" pad="P$1"/>
+<wire x1="76.2" y1="19.05" x2="87.63" y2="13.97" width="0" layer="19" extent="1-1"/>
 </signal>
 </signals>
@@
 </note>
 <note version="8.2" severity="warning">
-Since Version 8.2, Eagle supports online libraries. The ids
+Since Version 8.2, EAGLE supports online libraries. The ids
 of those online libraries will not be understood (or retained)
 with this version.
