File: AMineralFire/MineralFire-0.3-smd-inprogress.sch (EAGLE design)
At the start: 86 parts, among them IC3 LM358D, Q1 20MHz, Q2 20MHz, Q3 MMBT3906LT1SMD, Q4 MMBT3906LT1SMD, Q5 MMBT3906LT1SMD, Q6 MMBT3906LT1SMD, Q7 MMBT3906LT1SMD, Q8 MMBT3906LT1SMD, Q9 MMBT3906LT1SMD, T1 200mA/40V, T2 200mA/40V, T3 200mA/40V, T4 200mA/40V, T5 200mA/40V, U1 ATMEGA328P_TQFP, U3 +12v, U4 ATMEGA328P_TQFP

Commit message: Updated design to use rotary encoder
Parts:
- removed MODESW1, MODESW2, MODESW3, PROGSW: TOGGLE_ON_OFF_ON, INSTRUO:TOGGLE_ON_OFF_ON
- removed TESTGND: WIREPAD3,81/1,1, wirepad:WIREPAD3,81/1,1
- removed U3: +12v, SparkFun-IC-Power:V_REG_78XX7812
- added C15, C16, C17, C18: 10nF, SparkFun-Capacitors:10NF-0603-50V-10%
- added C20: 10u, rcl:CPOL-US153CLV-0505
- added ENC1, ENC2: ENCODER-2LED, SparkFun-Switches:ENCODER-2LED
- added R27, R38: 330, SparkFun-Resistors:330OHM-0603-1/10W-1%
- added U2, U5: 7805, INSTRUO:V-REG
- C7: value 10uF -> 10u
- R1, R10, R14, R4: value 1k -> 10k; device SparkFun-Resistors:1KOHM-0603-1/10W-1% -> SparkFun-Resistors:10KOHM-0603-1/10W-1%
- R11, R12, R2, R20, R3, R5, R6: value 100k -> 10k; device SparkFun-Resistors:100KOHM-0603-1/10W-1% -> SparkFun-Resistors:10KOHM-0603-1/10W-1%
- R21: value 100k -> 330; device SparkFun-Resistors:100KOHM-0603-1/10W-1% -> SparkFun-Resistors:330OHM-0603-1/10W-1%
- R31: value 100 -> 330; device SparkFun-Resistors:100OHM-0603-1/10W-1% -> SparkFun-Resistors:330OHM-0603-1/10W-1%
Connections:
- net BUTLED renamed TRIG1
- removed net LBUTTON: BUT1G$1.1, BUT1G$1.3, R31.1, U1.ADC6
- removed net T1: MODESW2.S, R11.2, U1.PD5(T1)
- removed net T2: MODESW2.O, R12.2, U1.PD4(XCK/T0)
- removed net T3: MODESW1.S, R2.2, U1.PC2(ADC2)
- removed net T4: MODESW1.O, R3.2, U1.PC3(ADC3)
- removed net T5: MODESW3.S, R5.2, U1.PC0(ADC0)
- removed net T6: MODESW3.O, R6.2, U1.PC1(ADC1)
- removed net T7: PROGSW.O, R21.2, U1.PD6(AIN0)
- removed net T8: PROGSW.S, R20.2, U1.PD7(AIN1)
- new net +12V1: U2.IN
- new net +12V2: U5.IN
- new net 5VDISP: C20.+, C7.+, ISP2.VCC, Q5.E, Q6.E, Q7.E, Q8.E, Q9.E, U2.OUT, U4.AREF, U4.AVCC, U4.VCC@4, U5.OUT
- new net BUT1: ENC1.SW, U1.ADC6
- new net BUT2: ENC2.SW, U1.ADC7
- new net BUT3: BUT1G$1.1, BUT1G$1.3, R20.1, U1.PD0(RXD)
- new net B_TRIG1: R5.1
- new net B_TRIG2: R14.1
- new net ENC1-G: R27.2, U1.PC0(ADC0)
- new net ENC1-R: ENC1.+R, R21.1, R21.2, R31.1, U1.PC1(ADC1)
- new net ENC1_TERMA: C15.1, R3.2, U1.PD4(XCK/T0)
- new net ENC1_TERMB: C16.1, R4.2, U1.PD5(T1)
- new net ENC2-G: ENC2.+G, R38.2, U1.PC2(ADC2)
- new net ENC2-R: ENC2.+R, R31.2, U1.PC3(ADC3)
- new net ENC2_TERMA: C17.1, R11.2, U1.PD6(AIN0)
- new net ENC2_TERMB: C18.1, R12.2, U1.PD7(AIN1)
- new net GND1: C7.-, U2.GND
- new net GND2: C20.-, U5.GND
- new net N$27: ENC2.A, R10.1, R11.1
- new net N$28: ENC2.B, R12.1, R6.1
- new net N$29: BUT1G$1.2, BUT1G$1.4
- new net N$30: ENC1.+G, R27.1
- new net N$35: R38.1
- net +12V: no longer U3.IN
- net +5V: now also R10.2, R14.2, R2.2, R20.2, R5.2, R6.2; no longer C7.+, ISP2.VCC, Q5.E, Q6.E, Q7.E, Q8.E, Q9.E, R11.1, R12.1, R2.1, R20.1, R21.1, R3.1, R31.2, R5.1, R6.1, U3.OUT, U4.AREF, U4.AVCC, U4.VCC@4
- net GND: now also C15.2, C16.2, C17.2, C18.2, ENC1.-, ENC2.-; no longer BUT1G$1.2, BUT1G$1.4, C7.-, R1.2, R10.2, R14.2, R4.2, TESTGND.P, U3.GND
- net N$12: now also ENC1.B, R1.1, R4.1; no longer MODESW2.P, R10.1
- net N$3: now also ENC1.C, ENC2.C; no longer MODESW1.P, R1.1
- net N$4: now also R1.2; no longer MODESW3.P, R4.1
- net N$6: now also ENC1.A, R2.1, R3.1; no longer PROGSW.P, R14.1

Commit message: Fixed routing errors
Parts:
- removed C9: 0.1uF, SparkFun-Capacitors:0.1UF-0603-100V-10%
Connections:
- removed net +12V: C4.+, C8.1, D1.C
- removed net +12V1: U2.IN
- removed net +12V2: U5.IN
- removed net -12V: C5.-, C9.2, D2.A
- removed net B_TRIG1: R5.1
- removed net B_TRIG2: R14.1
- removed net CS: U1.PB2(SS/OC1B)
- removed net GND1: C7.-, U2.GND
- removed net GND2: C20.-, U5.GND
- removed net N$25: C14.2
- removed net N$26: R34.2
- removed net N$29: BUT1G$1.2, BUT1G$1.4
- removed net N$4: R1.2
- new net 12V: C4.+, C8.1, D1.C, U2.IN, U5.IN
- new net 5V: C10.1, C11.1, C12.1, C7.+, IC3P.V+, ISP1.VCC, R1.2, R10.2, R14.2, R2.2, R36.1, R37.1, R5.2, R6.2, R7.2, R9.2, U1.AREF, U1.AVCC, U1.VCC@4, U2.OUT
- new net N$36: ENC2.+R, R31.1
- new net N$38: C5.-, D2.A
- net +5V: no longer C10.1, C11.1, C12.1, IC3P.V+, ISP1.VCC, R10.2, R14.2, R2.2, R36.1, R37.1, R5.2, R6.2, R7.2, R9.2, U1.AREF, U1.AVCC, U1.VCC@4
- net 5VDISP: no longer C7.+, U2.OUT
- net BUT1: now also R5.1
- net BUT2: now also R14.1
- net ENC1-R: no longer ENC1.+R, R21.1, R31.1
- net ENC2-G: no longer ENC2.+G
- net ENC2-R: no longer ENC2.+R
- net GND: now also BUT1G$1.2, BUT1G$1.4, C20.-, C7.-, ENC1.C, ENC2.C, U2.GND, U5.GND; no longer C9.1
- net N$19: now also C14.2
- net N$22: now also R34.2
- net N$3: now also ENC1.+R, R21.1; no longer ENC1.C, ENC2.C
- net N$35: now also ENC2.+G
