File: AMineralFire/MineralFire-0.4-OLED-inprogress.sch (EAGLE design)
At the start: 62 parts, among them IC3 LM358D, Q1 20MHz, T1 200mA/40V, U1 ATMEGA328P_TQFP, U2 7805

Commit message: Towards OLED
Connections:
- new net CS-DISP: U1.PB2(SS/OC1B)
- new net DC-DISP: U1.PC4(ADC4/SDA)
- new net RST-DISP: U1.PC5(ADC5/SCL)
Changed lines of the file:
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@@
+</segment>
+</net>
+<net name="CS-DISP" class="0">
+<segment>
+<pinref part="U1" gate="U$1" pin="PB2(SS/OC1B)"/>
+<wire x1="111.76" y1="17.78" x2="114.3" y2="17.78" width="0.1524" layer="91"/>
+<label x="114.3" y="17.78" size="1.778" layer="95" xref="yes"/>
+</segment>
+</net>
+<net name="DC-DISP" class="0">
+<segment>
+<pinref part="U1" gate="U$1" pin="PC4(ADC4/SDA)"/>
+<wire x1="111.76" y1="58.42" x2="119.38" y2="58.42" width="0.1524" layer="91"/>
+<label x="119.38" y="58.42" size="1.778" layer="95" xref="yes"/>
+</segment>
+</net>
+<net name="RST-DISP" class="0">
+<segment>
+<pinref part="U1" gate="U$1" pin="PC5(ADC5/SCL)"/>
+<wire x1="111.76" y1="55.88" x2="119.38" y2="55.88" width="0.1524" layer="91"/>
+<label x="119.38" y="55.88" size="1.778" layer="95" xref="yes"/>
+<label x="119.38" y="55.88" size="1.778" layer="95" xref="yes"/>
 </segment>
 </net>

Commit message: trying connector for oled
Parts:
- added J1: (no value), SparkFun-Connectors:CONN_07LOCK
Connections:
- net 5V: now also J1.2
- net CS-DISP: now also J1.7
- net DC-DISP: now also J1.6
- net GND: now also J1.1
- net MOSI: now also J1.4
- net RST-DISP: now also J1.5
- net SCK: now also J1.3
Other:
- note added: "CS"
- note added: "GND"
Changed lines of the file:
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@@
 <part name="U2" library="INSTRUO" deviceset="V-REG" device="" value="7805"/>
 <part name="C7" library="rcl" deviceset="CPOL-US" device="153CLV-0505" value="10u"/>
+<part name="J1" library="SparkFun-Connectors" library_urn="urn:adsk.eagle:library:513" deviceset="CONN_07" device="LOCK" package3d_urn="urn:adsk.eagle:package:38132/1"/>
 </parts>
 <sheets>
@@
 <description>Display</description>
 <plain>
+<text x="38.1" y="55.88" size="1.778" layer="91" rot="MR0">GND</text>
+<text x="38.1" y="76.2" size="1.778" layer="91" rot="MR0">CS</text>
 </plain>
 <instances>
+<instance part="J1" gate="G$1" x="35.56" y="63.5"/>
 </instances>
 <busses>
 </busses>
 <nets>
+<net name="DC-DISP" class="0">
+<segment>
+<pinref part="J1" gate="G$1" pin="6"/>
+<wire x1="40.64" y1="71.12" x2="45.72" y2="71.12" width="0.1524" layer="91"/>
+<label x="45.72" y="71.12" size="1.778" layer="95" xref="yes"/>
+</segment>
+</net>
+<net name="RST-DISP" class="0">
+<segment>
+<pinref part="J1" gate="G$1" pin="5"/>
+<wire x1="40.64" y1="68.58" x2="45.72" y2="68.58" width="0.1524" layer="91"/>
+<label x="45.72" y="68.58" size="1.778" layer="95" xref="yes"/>
+</segment>
+</net>
+<net name="MOSI" class="0">
+<segment>
+<pinref part="J1" gate="G$1" pin="4"/>
+<wire x1="40.64" y1="66.04" x2="45.72" y2="66.04" width="0.1524" layer="91"/>
+<label x="45.72" y="66.04" size="1.778" layer="95" xref="yes"/>
+</segment>
+</net>
+<net name="5V" class="0">
+<segment>
+<pinref part="J1" gate="G$1" pin="2"/>
+<wire x1="40.64" y1="60.96" x2="45.72" y2="60.96" width="0.1524" layer="91"/>
+<label x="45.72" y="60.96" size="1.778" layer="95" xref="yes"/>
+</segment>
+</net>
+<net name="GND" class="1">
+<segment>
+<pinref part="J1" gate="G$1" pin="1"/>
+<wire x1="40.64" y1="58.42" x2="45.72" y2="58.42" width="0.1524" layer="91"/>
+<label x="45.72" y="58.42" size="1.778" layer="95" xref="yes"/>
+</segment>
+</net>
+<net name="SCK" class="0">
+<segment>
+<pinref part="J1" gate="G$1" pin="3"/>
+<wire x1="40.64" y1="63.5" x2="45.72" y2="63.5" width="0.1524" layer="91"/>
+<label x="45.72" y="63.5" size="1.778" layer="95" xref="yes"/>
+</segment>
+</net>
+<net name="CS-DISP" class="0">
+<segment>
+<pinref part="J1" gate="G$1" pin="7"/>
+<wire x1="40.64" y1="73.66" x2="45.72" y2="73.66" width="0.1524" layer="91"/>
+<label x="45.72" y="73.66" size="1.778" layer="95" xref="yes"/>
+</segment>
+</net>
 </nets>
 </sheet>

Commit message: upadted
Parts:
- removed J1: (no value), SparkFun-Connectors:CONN_07LOCK
- added IC1: 74AC32D, 74xx-eu:74AC32D
- added IC2: 74AC86D, 74xx-eu:74AC86D
- added JP1: (no value), Adafruit_1.3_128x64_OLED:MICROBUILDER_HEADER-1X8ROUND
- C3: value 10u -> 10uF
- renumbered C7 to C3
Connections:
- removed net B_TRIG: BUTG$1.1, BUTG$1.3, R9.1, U1.PD3(INT1)
- new net BUT4: BUTG$1.1, BUTG$1.3, R9.1, U1.PD1(TXD)
- new net ENC_INT: IC2A.O, U1.PD3(INT1)
- new net N$4: IC1A.O, IC2A.I0
- new net N$5: IC1B.O, IC2A.I1
- net 5V: now also IC1P.VCC, IC2P.VCC, JP1.2; no longer J1.2
- net CS-DISP: now also JP1.7; no longer J1.7
- net DC-DISP: now also JP1.6; no longer J1.6
- net ENC1_TERMA: now also IC1A.I0
- net ENC1_TERMB: now also IC1A.I1
- net ENC2_TERMA: now also IC1B.I0
- net ENC2_TERMB: now also IC1B.I1
- net GND: now also IC1P.GND, IC2P.GND, JP1.1; no longer J1.1
- net MOSI: now also JP1.4; no longer J1.4
- net RST-DISP: now also JP1.5; no longer J1.5
- net SCK: now also JP1.3; no longer J1.3
